File: Main_Board.sch (KiCad schematic (older format))
At the start: 50 parts, among them J1 DB9_Female, J2 Conn_01x07_Female, Q1 Q_PNP_BCE, Q2 Q_NPN_BCE

Commit message: Connections
Parts:
- removed J2: Conn_01x07_Female, symbol Connector:Conn_01x07_Female
- added J?: SAMTEC-DW-12-07-X-S-200, SAMTEC-DW-12-07-X-S-200, symbol SAMTEC-DW-12-07-X-S-200:SAMTEC-DW-12-07-X-S-200
Connections:
- wire segments 201 -> 194
Other:
- moved on the sheet: -3V1, -5V1, C10, C12, C8, C9, R14, R15, R19, R20

Commit message: I/O
Parts:
- removed J1: DB9_Female, DG-9:TE_1-1634580-2, symbol Connector:DB9_Female
- added GND, Vin, data_in, data_out: TestPoint, TestPoint:TestPoint_Plated_Hole_D2.0mm, symbol Connector:TestPoint
- added J?: SAMTEC-DW-12-07-X-S-200, SAMTEC-DW-12-07-X-S-200, symbol SAMTEC-DW-12-07-X-S-200:SAMTEC-DW-12-07-X-S-200
Connections:
- net GND: now also GND.1
- net Vin: now also Vin.1
- new net Din: data_in.1
- new net Dout: data_out.1
- no-connect marks 7 -> 0
Other:
- moved on the sheet: J?
Changed lines of the file:
@@
 Wire Wire Line
 	8200 1850 8750 1850
-$Comp
-L power:GND #PWR0109
-U 1 1 5DD484BF
-P 1350 7250
-F 0 "#PWR0109" H 1350 7000 50  0001 C CNN
-F 1 "GND" H 1355 7077 50  0000 C CNN
-F 2 "" H 1350 7250 50  0001 C CNN
-F 3 "" H 1350 7250 50  0001 C CNN
-	1    1350 7250
-	1    0    0    -1
-$EndComp
-NoConn ~ 1350 7150
-NoConn ~ 1350 7050
-NoConn ~ 1350 6950
-NoConn ~ 1350 6850
-NoConn ~ 1350 6750
-NoConn ~ 1350 6650
-NoConn ~ 1350 6550
-Text Label 1350 6450 0    50   ~ 0
-Vin
-$Comp
-L Connector:DB9_Female J1
-U 1 1 5DD00653
-P 1050 6850
-F 0 "J1" H 968 6158 50  0000 C CNN
-F 1 "DB9_Female" H 968 6249 50  0000 C CNN
-F 2 "DG-9:TE_1-1634580-2" H 1050 6850 50  0001 C CNN
-F 3 " ~" H 1050 6850 50  0001 C CNN
-	1    1050 6850
-	-1   0    0    1
-$EndComp
 Wire Wire Line
 	3900 4700 4100 4700
@@
 L SAMTEC-DW-12-07-X-S-200:SAMTEC-DW-12-07-X-S-200 J?
 U 1 1 5E451443
-P 10100 2750
-F 0 "J?" H 10000 3050 50  0000 L CNN
-F 1 "SAMTEC-DW-12-07-X-S-200" H 10000 3150 50  0000 L CNN
-F 2 "SAMTEC-DW-12-07-X-S-200" H 10100 2750 50  0001 L BNN
-F 3 "" H 10100 2750 50  0001 C CNN
-	1    10100 2750
-	1    0    0    -1
-$EndComp
+P 10000 1150
+F 0 "J?" H 9900 1450 50  0000 L CNN
+F 1 "SAMTEC-DW-12-07-X-S-200" H 9900 1550 50  0000 L CNN
+F 2 "SAMTEC-DW-12-07-X-S-200" H 10000 1150 50  0001 L BNN
+F 3 "" H 10000 1150 50  0001 C CNN
+	1    10000 1150
+	1    0    0    -1
+$EndComp
+$Comp
+L SAMTEC-DW-12-07-X-S-200:SAMTEC-DW-12-07-X-S-200 J?
+U 1 1 5E48B8C7
+P 10000 3350
+F 0 "J?" H 9900 3650 50  0000 L CNN
+F 1 "SAMTEC-DW-12-07-X-S-200" H 9900 3750 50  0000 L CNN
+F 2 "SAMTEC-DW-12-07-X-S-200" H 10000 3350 50  0001 L BNN
+F 3 "" H 10000 3350 50  0001 C CNN
+	1    10000 3350
+	1    0    0    -1
+$EndComp
+$Comp
+L Connector:TestPoint Vin
+U 1 1 5E48CCC4
+P 10150 5550
+F 0 "Vin" H 10208 5668 50  0000 L CNN
+F 1 "TestPoint" H 10208 5577 50  0000 L CNN
+F 2 "TestPoint:TestPoint_Plated_Hole_D2.0mm" H 10350 5550 50  0001 C CNN
+F 3 "~" H 10350 5550 50  0001 C CNN
+	1    10150 5550
+	1    0    0    -1
+$EndComp
+$Comp
+L Connector:TestPoint GND
+U 1 1 5E48DDB9
+P 10700 5550
+F 0 "GND" H 10758 5668 50  0000 L CNN
+F 1 "TestPoint" H 10758 5577 50  0000 L CNN
+F 2 "TestPoint:TestPoint_Plated_Hole_D2.0mm" H 10900 5550 50  0001 C CNN
+F 3 "~" H 10900 5550 50  0001 C CNN
+	1    10700 5550
+	1    0    0    -1
+$EndComp
+$Comp
+L Connector:TestPoint data_out
+U 1 1 5E48E098
+P 10700 5950
+F 0 "data_out" H 10758 6068 50  0000 L CNN
+F 1 "TestPoint" H 10758 5977 50  0000 L CNN
+F 2 "TestPoint:TestPoint_Plated_Hole_D2.0mm" H 10900 5950 50  0001 C CNN
+F 3 "~" H 10900 5950 50  0001 C CNN
+	1    10700 5950
+	1    0    0    -1
+$EndComp
+$Comp
+L Connector:TestPoint data_in
+U 1 1 5E48E2AA
+P 10150 5950
+F 0 "data_in" H 10208 6068 50  0000 L CNN
+F 1 "TestPoint" H 10208 5977 50  0000 L CNN
+F 2 "TestPoint:TestPoint_Plated_Hole_D2.0mm" H 10350 5950 50  0001 C CNN
+F 3 "~" H 10350 5950 50  0001 C CNN
+	1    10150 5950
+	1    0    0    -1
+$EndComp
+$Comp
+L power:GND #PWR?
+U 1 1 5E4901A5
+P 10700 5550
+F 0 "#PWR?" H 10700 5300 50  0001 C CNN
+F 1 "GND" H 10705 5377 50  0000 C CNN
+F 2 "" H 10700 5550 50  0001 C CNN
+F 3 "" H 10700 5550 50  0001 C CNN
+	1    10700 5550
+	1    0    0    -1
+$EndComp
+Text Label 10150 5650 0    50   ~ 0
+Vin
+Wire Wire Line
+	10150 5550 10150 5650
+Wire Wire Line
+	10150 5950 10150 6050
+Wire Wire Line
+	10700 5950 10700 6050
+Text Label 10150 6050 0    50   ~ 0
+Din
+Text Label 10700 6050 0    50   ~ 0
+Dout
 $EndSCHEMATC

Commit message: I/O
Connections:
- net +15V: now also J?.1
Changed lines of the file:
@@
 Text Label 10700 6050 0    50   ~ 0
 Dout
+Text Label 9550 1150 0    50   ~ 0
++15V
+Text Label 9550 1250 0    50   ~ 0
++5V
+Text Label 9550 1350 0    50   ~ 0
++3V
+$Comp
+L power:GND #PWR?
+U 1 1 5E4B6CF3
+P 9650 1450
+F 0 "#PWR?" H 9650 1200 50  0001 C CNN
+F 1 "GND" H 9655 1277 50  0000 C CNN
+F 2 "" H 9650 1450 50  0001 C CNN
+F 3 "" H 9650 1450 50  0001 C CNN
+	1    9650 1450
+	0    1    1    0
+$EndComp
+Text Label 9550 1550 0    50   ~ 0
+-3V
+Text Label 9550 1650 0    50   ~ 0
+-5V
+Text Label 9550 1750 0    50   ~ 0
+-15V
+Wire Wire Line
+	9550 1150 9800 1150
 $EndSCHEMATC

Commit message: I/O
Parts:
- C10, C12, C8, C9: value 100u -> 10u
Changed lines of the file:
@@
 P 5150 3900
 F 0 "C8" H 5265 3946 50  0000 L CNN
-F 1 "100u" H 5265 3855 50  0000 L CNN
+F 1 "10u" H 5265 3855 50  0000 L CNN
 F 2 "Capacitor_SMD:C_0805_2012Metric" H 5188 3750 50  0001 C CNN
 F 3 "~" H 5150 3900 50  0001 C CNN
@@
 P 6550 3900
 F 0 "C9" H 6665 3946 50  0000 L CNN
-F 1 "100u" H 6665 3855 50  0000 L CNN
+F 1 "10u" H 6665 3855 50  0000 L CNN
 F 2 "Capacitor_SMD:C_0805_2012Metric" H 6588 3750 50  0001 C CNN
 F 3 "~" H 6550 3900 50  0001 C CNN
@@
 P 7450 3900
 F 0 "C10" H 7565 3946 50  0000 L CNN
-F 1 "100u" H 7565 3855 50  0000 L CNN
+F 1 "10u" H 7565 3855 50  0000 L CNN
 F 2 "Capacitor_SMD:C_0805_2012Metric" H 7488 3750 50  0001 C CNN
 F 3 "~" H 7450 3900 50  0001 C CNN
@@
 P 8850 3900
 F 0 "C12" H 8965 3946 50  0000 L CNN
-F 1 "100u" H 8965 3855 50  0000 L CNN
+F 1 "10u" H 8965 3855 50  0000 L CNN
 F 2 "Capacitor_SMD:C_0805_2012Metric" H 8888 3750 50  0001 C CNN
 F 3 "~" H 8850 3900 50  0001 C CNN

Commit message: Caps
Parts:
- added C?: 10u, Capacitor_SMD:C_0805_2012Metric, symbol Device:C
- added C?: 5u, Capacitor_SMD:C_0805_2012Metric, symbol Device:C
- C8: value 10u -> 5u
Connections:
- net GND: now also C?.1, C?.1
- net at -5V1.1 (ADJ), R14.2, R15.1: now also C?.2
- net at -3V1.1 (ADJ), R19.2, R20.1: now also C?.2
Changed lines of the file:
@@
 P 5150 3900
 F 0 "C8" H 5265 3946 50  0000 L CNN
-F 1 "10u" H 5265 3855 50  0000 L CNN
+F 1 "5u" H 5265 3855 50  0000 L CNN
 F 2 "Capacitor_SMD:C_0805_2012Metric" H 5188 3750 50  0001 C CNN
 F 3 "~" H 5150 3900 50  0001 C CNN
@@
 Wire Wire Line
 	9550 1150 9800 1150
+$Comp
+L Device:C C?
+U 1 1 5E43C68E
+P 5800 3600
+F 0 "C?" H 5915 3646 50  0000 L CNN
+F 1 "10u" H 5915 3555 50  0000 L CNN
+F 2 "Capacitor_SMD:C_0805_2012Metric" H 5838 3450 50  0001 C CNN
+F 3 "~" H 5800 3600 50  0001 C CNN
+	1    5800 3600
+	1    0    0    -1
+$EndComp
+Connection ~ 5800 3750
+$Comp
+L Device:C C?
+U 1 1 5E43CC18
+P 8100 3600
+F 0 "C?" H 8215 3646 50  0000 L CNN
+F 1 "5u" H 8215 3555 50  0000 L CNN
+F 2 "Capacitor_SMD:C_0805_2012Metric" H 8138 3450 50  0001 C CNN
+F 3 "~" H 8100 3600 50  0001 C CNN
+	1    8100 3600
+	1    0    0    -1
+$EndComp
+Connection ~ 8100 3750
+Wire Wire Line
+	8100 3350 8100 3450
+Wire Wire Line
+	5800 3350 5800 3450
 $EndSCHEMATC

Commit message: R
Parts:
- R14: value 360 -> 298
- R15, R20: value 120 -> 100
- R19: value 168 -> 140
Changed lines of the file:
@@
 P 6200 3500
 F 0 "R14" H 6270 3546 50  0000 L CNN
-F 1 "360" H 6270 3455 50  0000 L CNN
+F 1 "298" H 6270 3455 50  0000 L CNN
 F 2 "Resistor_SMD:R_0805_2012Metric" V 6130 3500 50  0001 C CNN
 F 3 "~" H 6200 3500 50  0001 C CNN
@@
 P 6200 4050
 F 0 "R15" H 6270 4096 50  0000 L CNN
-F 1 "120" H 6270 4005 50  0000 L CNN
+F 1 "100" H 6270 4005 50  0000 L CNN
 F 2 "Resistor_SMD:R_0805_2012Metric" V 6130 4050 50  0001 C CNN
 F 3 "~" H 6200 4050 50  0001 C CNN
@@
 P 8500 3500
 F 0 "R19" H 8570 3546 50  0000 L CNN
-F 1 "168" H 8570 3455 50  0000 L CNN
+F 1 "140" H 8570 3455 50  0000 L CNN
 F 2 "Resistor_SMD:R_0805_2012Metric" V 8430 3500 50  0001 C CNN
 F 3 "~" H 8500 3500 50  0001 C CNN
@@
 P 8500 4050
 F 0 "R20" H 8570 4096 50  0000 L CNN
-F 1 "120" H 8570 4005 50  0000 L CNN
+F 1 "100" H 8570 4005 50  0000 L CNN
 F 2 "Resistor_SMD:R_0805_2012Metric" V 8430 4050 50  0001 C CNN
 F 3 "~" H 8500 4050 50  0001 C CNN

Commit message: I/O
Connections:
- net +3V: now also J?.3
- net +5V: now also J?.2
- net -15V: now also J?.7
- net -3V: now also J?.5
- net -5V: now also J?.6
- net GND: now also J?.4
Changed lines of the file:
@@
 Wire Wire Line
 	5800 3350 5800 3450
+Wire Wire Line
+	9550 1250 9800 1250
+Wire Wire Line
+	9800 1350 9550 1350
+Wire Wire Line
+	9650 1450 9800 1450
+Wire Wire Line
+	9800 1550 9550 1550
+Wire Wire Line
+	9550 1650 9800 1650
+Wire Wire Line
+	9800 1750 9550 1750
 $EndSCHEMATC

Commit message: Caps
Parts:
- C10: value 10u -> 5u
- C?: value 5u -> 10u
Changed lines of the file:
@@
 P 7450 3900
 F 0 "C10" H 7565 3946 50  0000 L CNN
-F 1 "10u" H 7565 3855 50  0000 L CNN
+F 1 "5u" H 7565 3855 50  0000 L CNN
 F 2 "Capacitor_SMD:C_0805_2012Metric" H 7488 3750 50  0001 C CNN
 F 3 "~" H 7450 3900 50  0001 C CNN
@@
 P 8100 3600
 F 0 "C?" H 8215 3646 50  0000 L CNN
-F 1 "5u" H 8215 3555 50  0000 L CNN
+F 1 "10u" H 8215 3555 50  0000 L CNN
 F 2 "Capacitor_SMD:C_0805_2012Metric" H 8138 3450 50  0001 C CNN
 F 3 "~" H 8100 3600 50  0001 C CNN
