File: Main_Board.kicad_pcb (KiCad board)
At the start: 2 copper layers, 54 parts, among them J1 Conn_01x10_Male, J2 Conn_01x10_Male, Q1 Q_PNP_BCE, Q2 Q_NPN_BCE, U1 AD667

Commit message: Outline
Other:
- board outline added: 95 x 95 mm
Changed lines of the file:
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@@
   (general
     (thickness 1.6)
-    (drawings 8)
+    (drawings 12)
     (tracks 0)
     (zones 0)
@@
     (pad_to_mask_clearance 0)
     (aux_axis_origin 0 0)
+    (grid_origin 12 81)
     (visible_elements 7FFFFFFF)
     (pcbplotparams
@@
     )
   )
+  (gr_line (start 107 81) (end 12 81) (layer Edge.Cuts) (width 0.1))
+  (gr_line (start 107 176) (end 107 81) (layer Edge.Cuts) (width 0.1))
+  (gr_line (start 12 176) (end 107 176) (layer Edge.Cuts) (width 0.1))
+  (gr_line (start 12 81) (end 12 176) (layer Edge.Cuts) (width 0.1))
   (gr_line (start 107 81) (end 106 81) (layer F.SilkS) (width 0.15))
   (gr_line (start 107 176) (end 107 81) (layer F.SilkS) (width 0.15))

Commit message: Didn't work
Parts:
- removed RV1: 100, Resistor_SMD:R_1206_3216Metric_Pad1.42x1.75mm_HandSolder
Changed lines of the file:
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@@
     (tracks 0)
     (zones 0)
-    (modules 54)
+    (modules 53)
     (nets 69)
   )
@@
     (add_net "Net-(RV1-Pad2)")
   )
-  (module Resistor_SMD:R_1206_3216Metric_Pad1.42x1.75mm_HandSolder (layer F.Cu)
-    (at 52 37)
-    (descr "Resistor SMD 1206 (3216 Metric), square (rectangular) end terminal, IPC_7351 nominal with elongated pad for handsoldering. (Body size source: http://www.tortai-tech.com/upload/download/2011102023233369053.pdf), generated with kicad-footprint-generator")
-    (tags "resistor handsolder")
-    (attr smd)
-    (fp_text reference RV1 (at 0 -1.82) (layer F.SilkS)
-      (effects (font (size 1 1) (thickness 0.15)))
-    )
-    (fp_text value 100 (at 0 1.82) (layer F.Fab)
-      (effects (font (size 1 1) (thickness 0.15)))
-    )
-    (fp_text user %R (at 0 0) (layer F.Fab)
-      (effects (font (size 0.8 0.8) (thickness 0.12)))
-    )
-    (fp_line (start 2.45 1.12) (end -2.45 1.12) (layer F.CrtYd) (width 0.05))
-    (fp_line (start 2.45 -1.12) (end 2.45 1.12) (layer F.CrtYd) (width 0.05))
-    (fp_line (start -2.45 -1.12) (end 2.45 -1.12) (layer F.CrtYd) (width 0.05))
-    (fp_line (start -2.45 1.12) (end -2.45 -1.12) (layer F.CrtYd) (width 0.05))
-    (fp_line (start -0.602064 0.91) (end 0.602064 0.91) (layer F.SilkS) (width 0.12))
-    (fp_line (start -0.602064 -0.91) (end 0.602064 -0.91) (layer F.SilkS) (width 0.12))
-    (fp_line (start 1.6 0.8) (end -1.6 0.8) (layer F.Fab) (width 0.1))
-    (fp_line (start 1.6 -0.8) (end 1.6 0.8) (layer F.Fab) (width 0.1))
-    (fp_line (start -1.6 -0.8) (end 1.6 -0.8) (layer F.Fab) (width 0.1))
-    (fp_line (start -1.6 0.8) (end -1.6 -0.8) (layer F.Fab) (width 0.1))
-    (pad 2 smd roundrect (at 1.4875 0) (size 1.425 1.75) (layers F.Cu F.Paste F.Mask) (roundrect_rratio 0.175439)
-      (net 54 "Net-(RV1-Pad2)"))
-    (pad 1 smd roundrect (at -1.4875 0) (size 1.425 1.75) (layers F.Cu F.Paste F.Mask) (roundrect_rratio 0.175439)
-      (net 55 "Net-(RV1-Pad1)"))
-    (model ${KISYS3DMOD}/Resistor_SMD.3dshapes/R_1206_3216Metric.wrl
-      (at (xyz 0 0 0))
-      (scale (xyz 1 1 1))
-      (rotate (xyz 0 0 0))
-    )
-  )
   (module Capacitor_SMD:C_1206_3216Metric_Pad1.42x1.75mm_HandSolder (layer F.Cu)

Commit message: Finished main traces
Parts:
- moved R10 3.17 mm to (36.3, 166.9)
- moved C15 2.97 mm to (31.9, 120.1)
- moved +15V1 2.12 mm to (20.0, 120.3)
- moved C18 2.12 mm to (15.0, 117.4)
- moved R16 2.12 mm to (28.1, 129.3)
- moved R19 2.12 mm to (22.9, 129.3)
- moved R20 2.12 mm to (18.1, 129.3)
- moved C10 1.53 mm to (65.3, 168.4)
- moved C2 0.96 mm to (23.4, 149.1)
- turned R5 to 180 degrees
Routing:
- net /+15V: track 0.00 -> 116.4 mm, vias 0 -> 2
- net /-15V: track 0.00 -> 89.2 mm
- net Net-(D1-Pad1): track 0.00 -> 54.9 mm, vias 0 -> 2
- net Net-(+3V1-Pad2): track 0.00 -> 45.2 mm
- net Net-(D2-Pad1): track 0.00 -> 36.3 mm
- net /+5V: track 0.00 -> 33.2 mm, vias 0 -> 2
- net Net-(Q2-Pad1): track 0.00 -> 32.6 mm
- net /+3V: track 0.00 -> 26.4 mm, vias 0 -> 1
- net Net-(C2-Pad2): track 0.00 -> 24.7 mm
- net /-5V: track 0.00 -> 22.2 mm
- net /-3V: track 0.00 -> 20.5 mm
- net Net-(+15V1-Pad2): track 0.00 -> 20.3 mm
- net Net-(-5V1-Pad1): track 0.00 -> 20.3 mm
- net Net-(-3V1-Pad1): track 0.00 -> 20.3 mm
- net /Vin: track 0.00 -> 20.2 mm
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
Commit message: Update
Parts:
- moved D1 5.30 mm to (39.1, 139.7)
- moved -15V1 5.30 mm to (23.9, 139.7)
- moved D2 5.30 mm to (21.7, 159.0)
- moved R2 5.30 mm to (22.7, 149.1)
- moved R3 5.30 mm to (18.7, 143.1)
- moved R4 5.30 mm to (27.7, 149.0)
- moved C2 5.30 mm to (18.1, 149.1)
- moved C8 5.30 mm to (34.7, 145.9)
- moved L1 5.30 mm to (33.8, 151.1)
- moved Q1 5.30 mm to (40.7, 154.0)
- moved R1 5.30 mm to (33.8, 157.0)
Routing:
- net /-15V: track 89.2 -> 63.1 mm
- net Net-(D2-Pad1): track 36.3 -> 24.8 mm
- net Net-(-15V1-Pad9): track 8.54 -> 0.00 mm
- net Net-(D1-Pad1): track 54.9 -> 49.8 mm, vias 2 -> 3
- net Net-(Q1-Pad2): track 18.8 -> 17.5 mm
- net Net-(C2-Pad2): track 24.7 -> 25.8 mm, vias 0 -> 2

Commit message: Update
Parts:
- moved -5V1 5.38 mm to (70.7, 169.1)
- moved C14 5.38 mm to (64.8, 159.1)
- moved R14 5.38 mm to (71.7, 149.8)
- moved R15 5.38 mm to (71.8, 159.1)
- moved C12 5.38 mm to (71.7, 154.8)
- moved C10 4.40 mm to (60.9, 168.3)
- moved -3V1 3.71 mm to (53.6, 169.1)
- moved C16 3.71 mm to (41.4, 168.1)
- moved C19 3.71 mm to (47.5, 159.9)
- moved R17 3.71 mm to (54.4, 149.8)
- moved R18 3.71 mm to (54.4, 159.9)
- moved C17 3.71 mm to (54.5, 154.8)
Routing:
- net /-15V: track 63.1 -> 79.2 mm

Commit message: Everything but ground
Routing:
- net Net-(-15V1-Pad9): track 0.00 -> 12.1 mm
- net /+15V: track 116.4 -> 115.6 mm
Changed lines of the file:
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@@
     (thickness 1.6)
     (drawings 12)
-    (tracks 212)
+    (tracks 214)
     (zones 0)
     (modules 53)
@@
   (segment (start 18.65 96.2) (end 17.9 96.2) (width 0.25) (layer F.Cu) (net 19))
   (segment (start 23.875 129.3) (end 26.675 132.1) (width 0.25) (layer F.Cu) (net 20))
-  (segment (start 26.675 132.1) (end 30.3 132.1) (width 0.25) (layer F.Cu) (net 20))
-  (segment (start 30.3 132.1) (end 31.4 131) (width 0.25) (layer F.Cu) (net 20))
-  (segment (start 31.4 131) (end 31.4 125.86) (width 0.25) (layer F.Cu) (net 20))
   (segment (start 25.55 167) (end 25.7 166.85) (width 0.25) (layer F.Cu) (net 20))
   (segment (start 20 167) (end 25.55 167) (width 0.25) (layer F.Cu) (net 20))
@@
   (segment (start 30.17 118.17) (end 30.17 124.63) (width 0.25) (layer B.Cu) (net 20))
   (segment (start 26.3 114.3) (end 30.17 118.17) (width 0.25) (layer B.Cu) (net 20))
-  (segment (start 31.4 125.86) (end 30.17 124.63) (width 0.25) (layer F.Cu) (net 20))
   (segment (start 30.17 124.63) (end 25.84 120.3) (width 0.25) (layer F.Cu) (net 20))
   (segment (start 19.216333 118.583667) (end 16.5 121.3) (width 0.25) (layer F.Cu) (net 20))
@@
   (segment (start 15 138.175) (end 15 170.125) (width 0.25) (layer F.Cu) (net 20))
   (segment (start 23.875 129.3) (end 15 138.175) (width 0.25) (layer F.Cu) (net 20))
+  (segment (start 30.17 124.63) (end 31 125.46) (width 0.25) (layer F.Cu) (net 20))
+  (segment (start 31 125.46) (end 31 130.5) (width 0.25) (layer F.Cu) (net 20))
+  (segment (start 29.4 132.1) (end 26.675 132.1) (width 0.25) (layer F.Cu) (net 20))
+  (segment (start 31 130.5) (end 29.4 132.1) (width 0.25) (layer F.Cu) (net 20))
   (segment (start 37.7875 166.9) (end 43.4 161.2875) (width 0.25) (layer F.Cu) (net 21))
   (segment (start 37.2 166.9) (end 37.7875 166.9) (width 0.25) (layer F.Cu) (net 21))
@@
   (segment (start 35.116333 95.716333) (end 40.55767 95.716333) (width 0.25) (layer F.Cu) (net 32))
   (segment (start 32.5 93.1) (end 35.116333 95.716333) (width 0.25) (layer F.Cu) (net 32))
+  (segment (start 32.850585 130) (end 25.92767 136.922915) (width 0.25) (layer F.Cu) (net 33))
+  (segment (start 35.125 130) (end 32.850585 130) (width 0.25) (layer F.Cu) (net 33))
   (segment (start 35.65 139.7) (end 29.75 139.7) (width 0.25) (layer F.Cu) (net 34))
   (segment (start 37.15 139.7) (end 35.65 139.7) (width 0.25) (layer F.Cu) (net 34))

Commit message: Traces
Routing:
- net /+15V: track 115.6 -> 87.5 mm, vias 2 -> 0
- net /+5V: track 33.2 -> 7.94 mm, vias 2 -> 0
- net /+3V: track 26.4 -> 13.6 mm, vias 1 -> 0
- net /Vin: track 20.2 -> 25.9 mm
Changed lines of the file:
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@@
     (thickness 1.6)
     (drawings 12)
-    (tracks 214)
+    (tracks 193)
     (zones 0)
     (modules 53)
@@
   (segment (start 47.440997 90.125) (end 45.28233 92.283667) (width 0.25) (layer F.Cu) (net 6))
   (segment (start 52 90.125) (end 47.440997 90.125) (width 0.25) (layer F.Cu) (net 6))
+  (segment (start 24.221578 117.522915) (end 25.28233 118.583667) (width 0.25) (layer B.Cu) (net 6))
+  (segment (start 23.82233 117.522915) (end 24.221578 117.522915) (width 0.25) (layer B.Cu) (net 6))
+  (segment (start 24.221578 91.222915) (end 25.28233 92.283667) (width 0.25) (layer B.Cu) (net 6))
+  (segment (start 23.82233 91.222915) (end 24.221578 91.222915) (width 0.25) (layer B.Cu) (net 6))
+  (segment (start 44.221578 91.222915) (end 45.28233 92.283667) (width 0.25) (layer B.Cu) (net 6))
+  (segment (start 43.82233 91.222915) (end 44.221578 91.222915) (width 0.25) (layer B.Cu) (net 6))
   (via (at 38.3 157.6) (size 0.8) (drill 0.4) (layers F.Cu B.Cu) (net 7))
   (segment (start 38.3 157.6) (end 38.3 145.5) (width 0.25) (layer B.Cu) (net 7))
@@
   (segment (start 28 165.6) (end 28 166.85) (width 0.25) (layer F.Cu) (net 8))
   (segment (start 25.1 162.7) (end 28 165.6) (width 0.25) (layer F.Cu) (net 8))
-  (segment (start 40 94) (end 38.95 94) (width 0.25) (layer F.Cu) (net 18))
-  (via (at 36.2 94) (size 0.8) (drill 0.4) (layers F.Cu B.Cu) (net 18))
-  (segment (start 38.95 94) (end 36.2 94) (width 0.25) (layer F.Cu) (net 18))
-  (segment (start 36.2 94.565685) (end 40.834315 99.2) (width 0.25) (layer B.Cu) (net 18))
-  (segment (start 36.2 94) (end 36.2 94.565685) (width 0.25) (layer B.Cu) (net 18))
-  (segment (start 40.834315 99.2) (end 47.6 99.2) (width 0.25) (layer B.Cu) (net 18))
-  (via (at 50.3 96.6) (size 0.8) (drill 0.4) (layers F.Cu B.Cu) (net 18))
-  (segment (start 47.6 99.2) (end 50.2 96.6) (width 0.25) (layer B.Cu) (net 18))
-  (segment (start 50.2 96.6) (end 50.3 96.6) (width 0.25) (layer B.Cu) (net 18))
-  (segment (start 50.3 96.6) (end 50.3 95.6) (width 0.25) (layer F.Cu) (net 18))
-  (segment (start 50.3 95.6) (end 48.7 94) (width 0.25) (layer F.Cu) (net 18))
-  (segment (start 48.7 94) (end 45.84 94) (width 0.25) (layer F.Cu) (net 18))
-  (segment (start 37.016333 92.283667) (end 40.55767 92.283667) (width 0.25) (layer F.Cu) (net 18))
-  (segment (start 36.2 94) (end 36.2 93.1) (width 0.25) (layer F.Cu) (net 18))
-  (segment (start 36.2 93.1) (end 37.016333 92.283667) (width 0.25) (layer F.Cu) (net 18))
+  (segment (start 40.55767 93.44233) (end 40 94) (width 0.25) (layer B.Cu) (net 18))
+  (segment (start 40.55767 92.283667) (end 40.55767 93.44233) (width 0.25) (layer B.Cu) (net 18))
+  (segment (start 42.274003 94) (end 45.84 94) (width 0.25) (layer B.Cu) (net 18))
+  (segment (start 40.55767 92.283667) (end 42.274003 94) (width 0.25) (layer B.Cu) (net 18))
   (segment (start 29.875 94) (end 31 95.125) (width 0.25) (layer F.Cu) (net 19))
   (segment (start 25.84 94) (end 29.875 94) (width 0.25) (layer F.Cu) (net 19))
-  (segment (start 19.709142 92.283667) (end 19.692809 92.3) (width 0.25) (layer F.Cu) (net 19))
-  (segment (start 20.55767 92.283667) (end 19.709142 92.283667) (width 0.25) (layer F.Cu) (net 19))
-  (segment (start 19.692809 92.3) (end 18.2 92.3) (width 0.25) (layer F.Cu) (net 19))
-  (via (at 16.5 94.8) (size 0.8) (drill 0.4) (layers F.Cu B.Cu) (net 19))
-  (segment (start 18.2 92.3) (end 16.5 94) (width 0.25) (layer F.Cu) (net 19))
-  (segment (start 16.5 94) (end 16.5 94.8) (width 0.25) (layer F.Cu) (net 19))
-  (segment (start 17.3 94) (end 25.84 94) (width 0.25) (layer B.Cu) (net 19))
-  (segment (start 16.5 94.8) (end 17.3 94) (width 0.25) (layer B.Cu) (net 19))
-  (segment (start 20 94.85) (end 18.65 96.2) (width 0.25) (layer F.Cu) (net 19))
-  (segment (start 20 94) (end 20 94.85) (width 0.25) (layer F.Cu) (net 19))
-  (segment (start 17.9 96.2) (end 16.5 94.8) (width 0.25) (layer F.Cu) (net 19))
-  (segment (start 18.65 96.2) (end 17.9 96.2) (width 0.25) (layer F.Cu) (net 19))
+  (segment (start 20 92.841337) (end 20.55767 92.283667) (width 0.25) (layer B.Cu) (net 19))
+  (segment (start 20 94) (end 20 92.841337) (width 0.25) (layer B.Cu) (net 19))
+  (segment (start 22.274003 94) (end 25.84 94) (width 0.25) (layer B.Cu) (net 19))
+  (segment (start 20.55767 92.283667) (end 22.274003 94) (width 0.25) (layer B.Cu) (net 19))
   (segment (start 23.875 129.3) (end 26.675 132.1) (width 0.25) (layer F.Cu) (net 20))
   (segment (start 25.55 167) (end 25.7 166.85) (width 0.25) (layer F.Cu) (net 20))
@@
   (segment (start 19.2 170.125) (end 15 170.125) (width 0.25) (layer F.Cu) (net 20))
   (segment (start 20 170.125) (end 19.2 170.125) (width 0.25) (layer F.Cu) (net 20))
-  (segment (start 18.95 120.3) (end 17.95 121.3) (width 0.25) (layer F.Cu) (net 20))
-  (segment (start 20 120.3) (end 18.95 120.3) (width 0.25) (layer F.Cu) (net 20))
-  (segment (start 17.95 121.3) (end 16.5 121.3) (width 0.25) (layer F.Cu) (net 20))
-  (via (at 16.5 121.3) (size 0.8) (drill 0.4) (layers F.Cu B.Cu) (net 20))
-  (segment (start 16.5 121.3) (end 16.5 117.6) (width 0.25) (layer B.Cu) (net 20))
-  (segment (start 16.5 117.6) (end 19.8 114.3) (width 0.25) (layer B.Cu) (net 20))
-  (segment (start 19.8 114.3) (end 26.3 114.3) (width 0.25) (layer B.Cu) (net 20))
-  (via (at 30.17 124.63) (size 0.8) (drill 0.4) (layers F.Cu B.Cu) (net 20))
-  (segment (start 30.17 118.17) (end 30.17 124.63) (width 0.25) (layer B.Cu) (net 20))
-  (segment (start 26.3 114.3) (end 30.17 118.17) (width 0.25) (layer B.Cu) (net 20))
   (segment (start 30.17 124.63) (end 25.84 120.3) (width 0.25) (layer F.Cu) (net 20))
-  (segment (start 19.216333 118.583667) (end 16.5 121.3) (width 0.25) (layer F.Cu) (net 20))
-  (segment (start 20.55767 118.583667) (end 19.216333 118.583667) (width 0.25) (layer F.Cu) (net 20))
   (segment (start 15 138.175) (end 15 170.125) (width 0.25) (layer F.Cu) (net 20))
   (segment (start 23.875 129.3) (end 15 138.175) (width 0.25) (layer F.Cu) (net 20))
@@
   (segment (start 29.4 132.1) (end 26.675 132.1) (width 0.25) (layer F.Cu) (net 20))
   (segment (start 31 130.5) (end 29.4 132.1) (width 0.25) (layer F.Cu) (net 20))
+  (segment (start 20 119.141337) (end 20.55767 118.583667) (width 0.25) (layer B.Cu) (net 20))
+  (segment (start 20 120.3) (end 20 119.141337) (width 0.25) (layer B.Cu) (net 20))
+  (segment (start 21.05 120.3) (end 25.84 120.3) (width 0.25) (layer B.Cu) (net 20))
+  (segment (start 20 120.3) (end 21.05 120.3) (width 0.25) (layer B.Cu) (net 20))
   (segment (start 37.7875 166.9) (end 43.4 161.2875) (width 0.25) (layer F.Cu) (net 21))
   (segment (start 37.2 166.9) (end 37.7875 166.9) (width 0.25) (layer F.Cu) (net 21))
@@
   (segment (start 19.5875 129.3) (end 22 129.3) (width 0.25) (layer F.Cu) (net 51))
   (segment (start 19 129.3) (end 19.5875 129.3) (width 0.25) (layer F.Cu) (net 51))
+  (segment (start 15 121.4) (end 16.216332 122.616332) (width 0.25) (layer F.Cu) (net 51))
+  (segment (start 15 118.3) (end 15 121.4) (width 0.25) (layer F.Cu) (net 51))
   (segment (start 19.957671 122.616332) (end 20.55767 122.016333) (width 0.25) (layer F.Cu) (net 51))
   (segment (start 16.216332 122.616332) (end 19.957671 122.616332) (width 0.25) (layer F.Cu) (net 51))
-  (segment (start 15 121.4) (end 16.216332 122.616332) (width 0.25) (layer F.Cu) (net 51))
-  (segment (start 15 118.3) (end 15 121.4) (width 0.25) (layer F.Cu) (net 51))
 )

Commit message: Grounddddddddddddd
Routing:
- net GND: track 0.00 -> 84.3 mm, vias 0 -> 1
- net Net-(+3V1-Pad2): track 45.2 -> 48.9 mm
Changed lines of the file:
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@@
     (thickness 1.6)
     (drawings 12)
-    (tracks 193)
+    (tracks 215)
     (zones 0)
     (modules 53)
@@
     (arrow2b (pts (xy 4 176) (xy 3.413579 174.873496)))
   )
+  (segment (start 23.91 138.541337) (end 24.46767 137.983667) (width 0.25) (layer B.Cu) (net 1))
+  (segment (start 23.91 139.7) (end 23.91 138.541337) (width 0.25) (layer B.Cu) (net 1))
+  (segment (start 27.475997 139.7) (end 29.19233 137.983667) (width 0.25) (layer B.Cu) (net 1))
+  (segment (start 23.91 139.7) (end 27.475997 139.7) (width 0.25) (layer B.Cu) (net 1))
+  (segment (start 28.131578 136.922915) (end 29.19233 137.983667) (width 0.25) (layer B.Cu) (net 1))
+  (segment (start 27.73233 136.922915) (end 28.131578 136.922915) (width 0.25) (layer B.Cu) (net 1))
+  (segment (start 25.28233 95.716333) (end 27.6 98.034003) (width 0.25) (layer F.Cu) (net 1))
+  (segment (start 27.6 98.034003) (end 27.634003 98.034003) (width 0.25) (layer F.Cu) (net 1))
+  (segment (start 19.0625 103) (end 19.0625 108) (width 0.25) (layer F.Cu) (net 1))
+  (segment (start 28.765997 99.2) (end 25.28233 95.716333) (width 0.25) (layer F.Cu) (net 1))
+  (segment (start 28.765997 105.234003) (end 28.765997 99.2) (width 0.25) (layer F.Cu) (net 1))
+  (segment (start 23.3 110.7) (end 28.765997 105.234003) (width 0.25) (layer F.Cu) (net 1))
+  (segment (start 19.0625 108) (end 21.7625 110.7) (width 0.25) (layer F.Cu) (net 1))
+  (segment (start 21.7625 110.7) (end 23.3 110.7) (width 0.25) (layer F.Cu) (net 1))
+  (via (at 28.6 86) (size 0.8) (drill 0.4) (layers F.Cu B.Cu) (net 1))
+  (segment (start 26.9375 86) (end 28.6 86) (width 0.25) (layer F.Cu) (net 1))
+  (segment (start 26.130858 95.716333) (end 25.28233 95.716333) (width 0.25) (layer B.Cu) (net 1))
+  (segment (start 28.6 93.247191) (end 26.130858 95.716333) (width 0.25) (layer B.Cu) (net 1))
+  (segment (start 28.6 86) (end 28.6 93.247191) (width 0.25) (layer B.Cu) (net 1))
+  (segment (start 25.28233 112.490005) (end 27.8 115.007675) (width 0.25) (layer B.Cu) (net 1))
+  (segment (start 25.28233 95.716333) (end 25.28233 112.490005) (width 0.25) (layer B.Cu) (net 1))
+  (segment (start 26.130858 122.016333) (end 25.28233 122.016333) (width 0.25) (layer B.Cu) (net 1))
+  (segment (start 27.8 120.347191) (end 26.130858 122.016333) (width 0.25) (layer B.Cu) (net 1))
+  (segment (start 27.8 115.007675) (end 27.8 120.347191) (width 0.25) (layer B.Cu) (net 1))
   (segment (start 18.656237 149.443763) (end 18.1 150) (width 0.25) (layer F.Cu) (net 2))
   (segment (start 19.12501 148.97499) (end 18.656237 149.443763) (width 0.25) (layer F.Cu) (net 2))
@@
   (segment (start 21.525 103) (end 25.0625 103) (width 0.25) (layer F.Cu) (net 27))
   (segment (start 20.9375 103) (end 21.525 103) (width 0.25) (layer F.Cu) (net 27))
-  (segment (start 19.957671 96.316332) (end 20.55767 95.716333) (width 0.25) (layer F.Cu) (net 28))
-  (segment (start 19.957671 108.524521) (end 19.957671 96.316332) (width 0.25) (layer F.Cu) (net 28))
-  (segment (start 20.45816 109.02501) (end 19.957671 108.524521) (width 0.25) (layer F.Cu) (net 28))
-  (segment (start 23.87499 109.02501) (end 20.45816 109.02501) (width 0.25) (layer F.Cu) (net 28))
-  (segment (start 31 97) (end 31 101.9) (width 0.25) (layer F.Cu) (net 28))
-  (segment (start 31 101.9) (end 23.87499 109.02501) (width 0.25) (layer F.Cu) (net 28))
-  (segment (start 15 97.9) (end 15 91.9375) (width 0.25) (layer F.Cu) (net 28))
-  (segment (start 15.8 98.7) (end 15 97.9) (width 0.25) (layer F.Cu) (net 28))
-  (segment (start 17.574003 98.7) (end 15.8 98.7) (width 0.25) (layer F.Cu) (net 28))
-  (segment (start 20.55767 95.716333) (end 17.574003 98.7) (width 0.25) (layer F.Cu) (net 28))
+  (segment (start 18.778833 95.716333) (end 15 91.9375) (width 0.25) (layer F.Cu) (net 28))
+  (segment (start 20.55767 95.716333) (end 18.778833 95.716333) (width 0.25) (layer F.Cu) (net 28))
+  (segment (start 31 97) (end 31 105) (width 0.25) (layer F.Cu) (net 28))
+  (segment (start 31 105) (end 24.2 111.8) (width 0.25) (layer F.Cu) (net 28))
+  (segment (start 24.2 111.8) (end 18.8 111.8) (width 0.25) (layer F.Cu) (net 28))
+  (segment (start 18.8 111.8) (end 16.4 109.4) (width 0.25) (layer F.Cu) (net 28))
+  (segment (start 16.4 99.874003) (end 20.55767 95.716333) (width 0.25) (layer F.Cu) (net 28))
+  (segment (start 16.4 109.4) (end 16.4 99.874003) (width 0.25) (layer F.Cu) (net 28))
   (segment (start 34.714585 91.222915) (end 42.01767 91.222915) (width 0.25) (layer F.Cu) (net 29))
   (segment (start 34 91.9375) (end 34.714585 91.222915) (width 0.25) (layer F.Cu) (net 29))
